Commit message: backup

File: wheeltec_robot_urdf/urdf/top_mec_dl_robot.urdf (robot description, URDF)
Before this commit: robot wheeltec_robot, 5 links, 4 joints
Links:
- added link laser; visual cylinder length=0.05 radius=0.04
Joints:
- added joint laser_joint: type fixed, parent base_link, child laser, origin xyz=0.275 0 0.245 rpy=0 0 0
